Commit message: fixes

File: example-package/urdf/robot_model.xacro (robot description, xacro)
@@ -6,5 +6,4 @@
     <xacro:include filename="$(find example-package)/urdf/wheel.xacro" />
     <xacro:include filename="$(find example-package)/urdf/inertial.xacro" />
-    <xacro:include filename="$(find example-package)/urdf/camera.xacro" />
     <link name="dummy_link"/>
     <joint name="dummy_joint" type="fixed">
@@ -54,5 +53,18 @@
         </visual>
     </link>
-    <xacro:camera x ="0.025" y="0.275" z="0.325"/>
+    <link name='camera_link'>
+        <visual name='camera_visual'>
+            <origin xyz="0 0 0" rpy=" 0 0 0"/>
+            <geometry>
+                <box size=".05 .05 .05"/>
+            </geometry>
+            <material name="blue"/>
+        </visual>
+    </link>
+    <joint type="fixed" name="camera_joint">
+        <origin xyz="0.025 0.275 0.325" rpy="0 0 ${pi/2}"/>
+        <child link="camera_link"/>
+        <parent link="base_link"/>
+    </joint>
     <xacro:wheel side="left" x="-0.325" y="0.15" z="0.1"/>
     <xacro:wheel side="right" x="0.325" y="0.15" z="0.1"/>

Commit message: fix gazebo rendering

File: example-package/urdf/robot_model.xacro (robot description, xacro)
@@ -6,9 +6,4 @@
     <xacro:include filename="$(find example-package)/urdf/wheel.xacro" />
     <xacro:include filename="$(find example-package)/urdf/inertial.xacro" />
-    <link name="dummy_link"/>
-    <joint name="dummy_joint" type="fixed">
-        <parent link="dummy_link"/>
-        <child link="base_link"/>
-    </joint>
     <link name='base_link'>
         <origin xyz="0.0 0.0 0.1" rpy="0.0 0 0.0"/>

Commit message: mount your package to container correctly

File: example-package/urdf/robot_model.xacro (robot description, xacro)
@@ -62,4 +62,18 @@
         <parent link="base_link"/>
     </joint>
+    <link name="lidar_link">
+            <visual name='lidar_visual'>
+                <origin xyz="0 0 0" rpy=" 0 0 0"/>
+                <geometry>
+                    <box size=".05 .05 .05"/>
+                </geometry>
+                <material name="red"/>
+            </visual>
+        </link>
+        <joint name="lidar_joint" type="fixed">
+            <origin xyz="-0.025 0.275 0.325" rpy="0 0 ${pi/2}"/>
+            <child link="lidar_link"/>
+            <parent link="base_link"/>
+        </joint>
     <xacro:wheel side="left" x="-0.325" y="0.15" z="0.1"/>
     <xacro:wheel side="right" x="0.325" y="0.15" z="0.1"/>
